Commit message: improved the model, world and other custom files. We worked on in the three of us together

File: src/my_robot_description/urdf/rubot/rubot_mecanum_custom.urdf (robot description, URDF)
Before this commit: robot rubot, 10 links, 9 joints
Joints:
- joint 3D_part_on_top_joint: origin xyz=-0.085 -0.1 0.01 rpy=0 0 3.14 -> xyz=-0.1 0.01 0.06 rpy=0 0 0
